Commit message: WIP: rack-pinion gripper 관련 설정 및 launch 파일 정리

File: src/army_manipulator_description/urdf/army_manipulator.urdf.xacro (robot description, xacro)
@@ -7,13 +7,9 @@
        meshes/{visual,collision}/*.stl 이 아직 없으므로 기본은 false로 두고,
        STL 파일을 받으면 use_mesh:=true 로 켜서 확인할 것. -->
-  <xacro:arg name="use_mesh" default="false"/>
-  <!-- 구동부 상면 높이: world -> base_link -->
-  <xacro:property name="base_height" value="0.350"/>
+  <xacro:arg name="use_mesh" default="true"/>
   <xacro:include filename="$(find army_manipulator_description)/urdf/materials.xacro"/>
   <xacro:include filename="$(find army_manipulator_description)/urdf/army_manipulator_ros2_control.xacro"/>
   <xacro:include filename="$(find army_manipulator_description)/urdf/army_manipulator_macro.xacro"/>
   <link name="world"/>
-  <xacro:army_manipulator prefix="" parent="world" use_mock_hardware="$(arg use_mock_hardware)" use_mesh="$(arg use_mesh)">
-    <origin xyz="0 0 ${base_height}" rpy="0 0 0"/>
-  </xacro:army_manipulator>
+  <xacro:army_manipulator prefix="" parent="world" use_mock_hardware="$(arg use_mock_hardware)" use_mesh="$(arg use_mesh)"/>
 </robot>

File: src/army_manipulator_description/urdf/army_manipulator_macro.xacro (robot description, xacro)
@@ -1,56 +1,48 @@
 <?xml version="1.0"?>
 <!--
-  MARU 로봇팔 매크로
+  MARU 로봇팔 매크로 (수정본)
   ============================================================
-  확정 파라미터 (베이스 상판 기준, prefix + parent 하위에 전개됨):
-    베이스→숄더 관절축 (sh_off)   = 106.6 mm
-    L1 숄더→엘보우                = 180 mm
-    L2 엘보우→리스트               = 220 mm
-    L3 리스트→TCP                 = 220 mm
-    Case C 조인트 오프셋 (z축):
-      shoulder_lift : -37.7 mm
-      elbow         : +18.8 mm
-      wrist         : -31.3 mm
-      gripper       : +38 mm
-  조인트 리미트:
-    기존에 이 파일에 하드코딩돼 있던 가정치(base ±180°, shoulder 0~120°,
-    elbow -90~+20°, wrist ±120°, gripper ±135° 등)는 전부 실측 인코더 기준
-    리미트로 대체되었다. 실제 <limit> 값은 config/joint_calibration.yaml의
-    raw_min/raw_max/zero_offset을 아래 보정식으로 계산해서 사용한다:
-      actual_joint_angle = raw_encoder_angle - zero_offset
-      actual_limit       = raw_limit         - zero_offset
-    zero_offset은 아직 실측 전이라 joint_calibration.yaml에 전부 0.0
-    placeholder로 들어있다(TODO(zero-offset)). 실측 후에는 그 yaml 파일만
-    갱신하면 되고, 이 xacro는 손댈 필요 없다.
-  TODO(home-pose): 각 조인트의 기본자세(홈 포지션, 현재는 SRDF group_state
-  "home"에서 전부 actual=0으로 둠)는 아직 CATIA 확인 전 플레이스홀더다.
-  TODO(base-pan-axis): base_rotate_joint의 회전축 방향/장착 orientation은
-  CATIA로 재확인 필요.
+  STL 좌표축 컨벤션 (모든 mesh에 공통, mesh 회전 없이 그대로 링크 로컬 프레임으로 사용):
+    전면부 = +Z, 하단부(바닥 방향) = +Y, 우측 = +X
+  즉 world_to_base가 무회전이므로 base_actuator 이하 모든 링크의 "Y축"이 곧
+  중력/수직 방향이고, "Z축"이 로봇의 전면(주 reach) 방향이다.
+  [오른손 법칙 검산 - 중요]
+  +X축 기준 양(+)의 회전(Rx(+θ))은 +Y축을 +Z축 쪽으로 돌린다. 즉 (0,1,0) -> (0,cosθ,sinθ).
+  뒤집어 말하면 +Z축은 -Y쪽으로 돈다: (0,0,1) -> (0,-sinθ,cosθ).
+  따라서 "전면(+Z)이 하단(+Y) 방향으로 숙여지는" 동작(카메라 하향 틸트 등)은
+  +X 회전이 아니라 X축 기준 음(-)의 회전이다. (이전 버전 주석은 부호 설명이 반대로
+  적혀 있었음 - 결론인 "하향 틸트 = -X 회전"은 맞았지만 근거 문장이 틀렸었다.)
+  같은 논리로, 어떤 링크의 "베이스 선회/pan"처럼 중력축(수직) 기준 회전이 필요한
+  조인트는 axis가 Y여야 하고(Z는 전면=수평축이라 pan에 쓰면 안 됨), 팔의 pitch류
+  조인트(shoulder/elbow/wrist)처럼 수평-좌우축 기준으로 앞뒤/상하로 숙이는 회전은
+  axis가 X여야 한다(좌우축이 곧 pitch 힌지축).
   ============================================================
 -->
 <robot xmlns:xacro="http://www.ros.org/wiki/xacro">
-  <xacro:macro name="army_manipulator" params="prefix parent use_mock_hardware:=true use_mesh:=false *origin">
-    <!-- ========== 치수 파라미터 ========== -->
-    <xacro:property name="sh_off"   value="0.1616"/>  <!-- base_link -> shoulder_pan_link -->
-    <xacro:property name="L1"       value="0.180"/>   <!-- shoulder -> elbow -->
-    <xacro:property name="L2"       value="0.220"/>   <!-- elbow -> wrist -->
-    <xacro:property name="L3"       value="0.220"/>   <!-- wrist -> tcp (gripper 포함) -->
-    <xacro:property name="off_shoulder" value="-0.0377"/>
+  <xacro:macro name="army_manipulator" params="prefix parent use_mock_hardware:=true use_mesh:=false">
+    <!-- ========== 치수 파라미터 (단위: m, 전부 STL 로컬 축 그대로) ========== -->
+    <xacro:property name="base_off"     value="0.04475"/>  <!-- base_actuator.stl Y-extent -->
+    <xacro:property name="shoulder_off" value="0.1039"/>  <!-- base_link.stl Y-extent -->
+    <xacro:property name="L1"           value="0.180"/>  <!-- shoulder_link.stl Y-extent -->
+    <xacro:property name="L2"           value="0.220"/>  <!-- elbow_link.stl Y-extent -->
+    <xacro:property name="L3"           value="0.150"/>  <!-- wrist_link.stl Y-extent -->
+    <xacro:property name="rack_off"     value="0.008"/>   <!-- pinion_gear -> rack_left/right (Z, 전면 깊이) -->
+    <xacro:property name="tcp_off"      value="0.065"/>   <!-- pinion_gear -> tcp_link (Z, 전면) -->
+    <!-- Case C 보조 오프셋: 전부 Z축(전면 방향) 성분. 팔의 주축 이동(-Y)과 항상
+         수직으로 별도 적용되는 소치수라서, 세 조인트(elbow/wrist/gripper) 모두
+         origin의 세 번째(Z) 자리에 들어가야 서로 같은 의미가 된다. -->
+    <xacro:property name="off_shoulder"  value="0.038"/>
     <xacro:property name="off_elbow"    value="0.0188"/>
     <xacro:property name="off_wrist"    value="-0.0313"/>
     <xacro:property name="off_gripper"  value="0.038"/>
-    <!-- ========== 관절 영점 보정(zero-offset) 리미트 ==========
-         config/joint_calibration.yaml의 raw_min/raw_max/zero_offset을 읽어
-         actual_limit = raw_limit - zero_offset 을 미리 계산해 둔다.
-         (xacro는 launch마다 새로 처리되므로, 이 yaml만 갱신하면 URDF 소스를
-         고치지 않아도 다음 실행부터 바로 반영된다.) -->
+    <!-- ========== 관절 영점 보정(zero-offset) 리미트 로드 ========== -->
     <xacro:arg name="joint_calibration_file"
                default="$(find army_manipulator_description)/config/joint_calibration.yaml"/>
     <xacro:property name="joint_calibration_file" value="$(arg joint_calibration_file)"/>
     <xacro:property name="joint_calib" value="${xacro.load_yaml(joint_calibration_file)}"/>
-    <xacro:property name="base_rotate_limit_lower"
-                     value="${joint_calib['joints']['base_rotate_joint']['raw_min'] - joint_calib['joints']['base_rotate_joint']['zero_offset']}"/>
-    <xacro:property name="base_rotate_limit_upper"
-                     value="${joint_calib['joints']['base_rotate_joint']['raw_max'] - joint_calib['joints']['base_rotate_joint']['zero_offset']}"/>
+    <xacro:property name="base_limit_lower"
+                     value="${joint_calib['joints']['base_joint']['raw_min'] - joint_calib['joints']['base_joint']['zero_offset']}"/>
+    <xacro:property name="base_limit_upper"
+                     value="${joint_calib['joints']['base_joint']['raw_max'] - joint_calib['joints']['base_joint']['zero_offset']}"/>
     <xacro:property name="shoulder_lift_limit_lower"
                      value="${joint_calib['joints']['shoulder_lift_joint']['raw_min'] - joint_calib['joints']['shoulder_lift_joint']['zero_offset']}"/>
@@ -69,21 +61,77 @@
     <xacro:property name="gripper_limit_upper"
                      value="${joint_calib['joints']['gripper_joint']['raw_max'] - joint_calib['joints']['gripper_joint']['zero_offset']}"/>
-    <!-- ========== parent -> base_link ========== -->
+    <!-- ========== parent -> base_actuator (fixed) ==========
+         [조인트] world(또는 상위 parent)와 무회전으로 연결. 즉 base_actuator의
+         로컬 X/Y/Z가 그대로 world의 우측/하단(중력)/전면이 된다. 이후 모든 링크의
+         축 해석 기준이 여기서 시작한다. -->
     <joint name="${prefix}world_to_base" type="fixed">
       <parent link="${parent}"/>
+      <child  link="${prefix}base_actuator"/>
+      <origin xyz="0 0 0" rpy="0 0 0"/>
+    </joint>
+    <!-- base_actuator: XH540-W270-T 모터 바디 (고정, world에 직접 마운트) -->
+    <link name="${prefix}base_actuator">
+      <xacro:if value="${use_mesh}">
+        <!-- [시각화] mesh는 STL 좌표축을 그대로 사용 (회전 없음). -->
+        <visual>
+          <origin xyz="0 0 0" rpy="0 0 0"/>
+          <geometry><mesh filename="package://army_manipulator_description/meshes/visual/base_actuator.stl" scale="0.001 0.001 0.001"/></geometry>
+          <material name="motor_dark"/>
+        </visual>
+        <!-- [콜리전] visual과 동일 회전. -->
+        <collision>
+          <origin xyz="0 0 0" rpy="0 0 0"/>
+          <geometry><mesh filename="package://army_manipulator_description/meshes/collision/base_actuator.stl" scale="0.001 0.001 0.001"/></geometry>
+        </collision>
+      </xacro:if>
+      <xacro:unless value="${use_mesh}">
+        <visual>
+          <origin xyz="0 0 0" rpy="0 0 0"/>
+          <geometry><cylinder radius="0.028" length="0.055"/></geometry>
+          <material name="motor_dark"/>
+        </visual>
+        <collision>
+          <origin xyz="0 0 0" rpy="0 0 0"/>
+          <geometry><cylinder radius="0.028" length="0.055"/></geometry>
+        </collision>
+      </xacro:unless>
+      <inertial>
+        <mass value="0.202"/>
+        <origin xyz="0 0 0"/>
+        <inertia ixx="1.3e-4" ixy="0" ixz="0" iyy="1.3e-4" iyz="0" izz="8.0e-5"/>
+      </inertial>
+    </link>
+    <!-- ========== base_actuator -> base_link (revolute, "베이스 선회") ==========
+         [조인트] 베이스 전체를 턴테이블처럼 수직축 기준으로 돌리는 조인트다.
+         world_to_base가 무회전이므로 이 링크의 Y축 = world의 중력(수직)축.
+         따라서 axis는 반드시 Y(0 1 0)여야 한다 - Z(전면)는 수평축이라 pan에 쓰면
+         팔이 옆으로 안 돌고 앞뒤로 텀블링하게 되므로 틀린 선택이었다. -->
+    <joint name="${prefix}base_joint" type="revolute">
+      <parent link="${prefix}base_actuator"/>
       <child  link="${prefix}base_link"/>
-      <xacro:insert_block name="origin"/>
-    </joint>
-    <!-- base_link: 암 마운팅 플레이트 (구동부 상면) -->
+      <origin xyz="0 0 0" rpy="0 0 0"/>
+      <axis xyz="0 0 1"/>
+      <limit lower="${base_limit_lower}" upper="${base_limit_upper}" effort="3.1" velocity="2.618"/>
+      <dynamics damping="0.05" friction="0.02"/>
+    </joint>
+    <!-- base_link: 베이스 회전판 -->
     <link name="${prefix}base_link">
-      <!-- mesh 파일은 사용자가 추후 추가 예정. scale은 CATIA(mm) -> URDF(m) 변환용. -->
-      <xacro:if value="${use_mesh}">
-        <visual>
-          <origin xyz="0 0 0" rpy="0 0 0"/>
+      <xacro:if value="${use_mesh}">
+        <!-- [시각화] X축 -90° 회전 + Z축 +9.08° 보정.
+             base_link.stl 삼각형 normal을 직접 계산해보면 원판 주면(제일 넓은
+             평면, ~27000mm^2)의 native normal이 (0.9874, 0, -0.1578)로 순수
+             +X에서 9.08° 벗어나 있다(STL 자체에 실제로 모델링된 tilt, 로딩/렌더링
+             아티팩트 아님). X축 -90° 적용 후에는 이 tilt가 XY평면 상의 편차로
+             나타나(rendered normal (0.9874,-0.1578,0)) 원판이 YZ평면에서 살짝
+             돌아가 보였다. Z축으로 +9.08°(atan2(0.1578,0.9874)) 추가 보정하면
+             정확히 (1,0,0)이 되어 원판이 YZ평면에 평평하게 눕는다. -->
+        <visual>
+          <origin xyz="0 0 0" rpy="${-pi/2} 0 0.15847"/>
           <geometry><mesh filename="package://army_manipulator_description/meshes/visual/base_link.stl" scale="0.001 0.001 0.001"/></geometry>
           <material name="petg_grey"/>
         </visual>
-        <collision>
-          <origin xyz="0 0 0" rpy="0 0 0"/>
+        <!-- [콜리전] visual과 동일 회전. -->
+        <collision>
+          <origin xyz="0 0 0" rpy="${-pi/2} 0 0.15847"/>
           <geometry><mesh filename="package://army_manipulator_description/meshes/collision/base_link.stl" scale="0.001 0.001 0.001"/></geometry>
         </collision>
@@ -103,78 +151,38 @@
         <mass value="0.3"/>
         <origin xyz="0 0 0"/>
-        <inertia ixx="2.5e-4" ixy="0" ixz="0"
-                 iyy="2.5e-4" iyz="0" izz="5.0e-4"/>
-      </inertial>
-    </link>
-    <!-- ========== base_link -> shoulder_pan_link ========== -->
-    <!-- XH540-W270-T | Z축 회전 (베이스 선회) -->
-    <joint name="${prefix}base_rotate_joint" type="revolute">
+        <inertia ixx="2.5e-4" ixy="0" ixz="0" iyy="2.5e-4" iyz="0" izz="5.0e-4"/>
+      </inertial>
+    </link>
+    <!-- ========== base_link -> shoulder_link (revolute, "숄더 피치") ==========
+         [조인트] 팔을 앞/뒤(전면-하단 평면)로 숙이는 pitch 조인트. 힌지축은
+         좌우(X) 수평축이어야 한다 - X는 중력축(Y)과도, 전면축(Z)과도 수직이라
+         "위아래로 숙이는" 회전에 정확히 들어맞는다. origin은 base_link.stl의
+         Y-extent(shoulder_off)만큼 +Z로 이동해 base_link 끝에 shoulder_link를
+         이어붙인다.
+         X축에는 off_gripper와 동일한 소치수 오프셋 적용.
+         [수정] 여기 있던 Z축 180° 반전을 제거했다 - shoulder/elbow/wrist 세
+         조인트에 각각 Z축 180°를 순서대로 넣으면 shoulder(180°)->elbow(0°,
+         상쇄)->wrist(180°)처럼 링크마다 번갈아 뒤집히면서 pitch 힌지축(X)
+         방향도 링크마다 반대가 돼버려 조인트 리밋 회전이 이상하게 보였다. -->
+    <joint name="${prefix}shoulder_lift_joint" type="revolute">
       <parent link="${prefix}base_link"/>
-      <child  link="${prefix}shoulder_pan_link"/>
-      <origin xyz="0 0 ${sh_off}" rpy="0 0 0"/>
-      <axis xyz="0 0 1"/>
-      <!-- 실측 인코더 리미트(raw_min/raw_max) - zero_offset. config/joint_calibration.yaml -->
-      <limit lower="${base_rotate_limit_lower}" upper="${base_rotate_limit_upper}"
-             effort="3.1" velocity="2.618"/>
-      <!-- XH540 stall torque 3.1 Nm @ 12V, no-load speed 25 RPM = 2.618 rad/s -->
-      <dynamics damping="0.05" friction="0.02"/>
-    </joint>
-    <!-- shoulder_pan_link: XH540 모터 바디 -->
-    <link name="${prefix}shoulder_pan_link">
-      <xacro:if value="${use_mesh}">
-        <visual>
-          <origin xyz="0 0 0" rpy="0 0 0"/>
-          <!-- base_actuator.stl = XH540-W270-T 모터 바디 (33.5x58.5x54.3mm 실측, XH540 규격과 일치) -->
-          <geometry><mesh filename="package://army_manipulator_description/meshes/visual/base_actuator.stl" scale="0.001 0.001 0.001"/></geometry>
-          <material name="motor_dark"/>
-        </visual>
-        <collision>
-          <origin xyz="0 0 0" rpy="0 0 0"/>
-          <geometry><mesh filename="package://army_manipulator_description/meshes/collision/base_actuator.stl" scale="0.001 0.001 0.001"/></geometry>
-        </collision>
-      </xacro:if>
-      <xacro:unless value="${use_mesh}">
-        <visual>
-          <origin xyz="0 0 0" rpy="0 0 0"/>
-          <geometry><cylinder radius="0.028" length="0.055"/></geometry>
-          <material name="motor_dark"/>
-        </visual>
-        <collision>
-          <origin xyz="0 0 0" rpy="0 0 0"/>
-          <geometry><cylinder radius="0.028" length="0.055"/></geometry>
-        </collision>
-      </xacro:unless>
-      <inertial>
-        <mass value="0.202"/>
-        <origin xyz="0 0 0"/>
-        <inertia ixx="1.3e-4" ixy="0" ixz="0"
-                 iyy="1.3e-4" iyz="0" izz="8.0e-5"/>
-      </inertial>
-    </link>
-    <!-- ========== shoulder_pan_link -> upper_arm_link ========== -->
-    <!-- RMD-X8-120 | Y축 회전 (숄더 피치), Case C 오프셋 z=-37.7mm -->
-    <joint name="${prefix}shoulder_lift_joint" type="revolute">
-      <parent link="${prefix}shoulder_pan_link"/>
-      <child  link="${prefix}upper_arm_link"/>
-      <origin xyz="0 0 ${off_shoulder}" rpy="0 0 0"/>
-      <axis xyz="0 1 0"/>
-      <!-- 실측 인코더 리미트(raw_min/raw_max) - zero_offset. config/joint_calibration.yaml -->
-      <limit lower="${shoulder_lift_limit_lower}" upper="${shoulder_lift_limit_upper}"
-             effort="120.0" velocity="1.047"/>
-      <!-- RMD-X8-120 peak torque 120 Nm, no-load speed ~10 RPM = 1.047 rad/s -->
+      <child  link="${prefix}shoulder_link"/>
+      <origin xyz="${off_gripper} 0 ${shoulder_off}" rpy="0 0 0"/>
+      <axis xyz="1 0 0"/>
+      <limit lower="${shoulder_lift_limit_lower}" upper="${shoulder_lift_limit_upper}" effort="120.0" velocity="1.047"/>
       <dynamics damping="1.0" friction="0.1"/>
     </joint>
-    <!-- upper_arm_link: CFRP 20x20x2T, L1 = 180mm -->
-    <link name="${prefix}upper_arm_link">
-      <xacro:if value="${use_mesh}">
-        <visual>
-          <origin xyz="0 0 0" rpy="0 0 0"/>
-          <!-- shoulder_link.stl = RMD-X8-120 출력 플랜지 + L1 CFRP 튜브 + RMD-X6-60 케이스 통합 파츠
-               (실측 Y span 260.1mm ≈ RMD-X8-120 플랜지 + L1(180mm) + RMD-X6-60 케이스 두께, 일치) -->
+    <!-- shoulder_link: RMD-X8-120 출력 플랜지 + L1 CFRP 튜브 + RMD-X6-60 케이스 통합 파츠 -->
+    <link name="${prefix}shoulder_link">
+      <xacro:if value="${use_mesh}">
+        <!-- [시각화] X축 -90° + Z축 180° 회전 적용. -->
+        <visual>
+          <origin xyz="0 0 0" rpy="${-pi/2} 0 ${pi}"/>
           <geometry><mesh filename="package://army_manipulator_description/meshes/visual/shoulder_link.stl" scale="0.001 0.001 0.001"/></geometry>
           <material name="cfrp"/>
         </visual>
-        <collision>
-          <origin xyz="0 0 0" rpy="0 0 0"/>
+        <!-- [콜리전] visual과 동일 회전. -->
+        <collision>
+          <origin xyz="0 0 0" rpy="${-pi/2} 0 ${pi}"/>
           <geometry><mesh filename="package://army_manipulator_description/meshes/collision/shoulder_link.stl" scale="0.001 0.001 0.001"/></geometry>
         </collision>
@@ -182,45 +190,46 @@
       <xacro:unless value="${use_mesh}">
         <visual>
-          <origin xyz="${L1/2} 0 0" rpy="0 1.5708 0"/>
+          <origin xyz="0 ${-L1/2} 0" rpy="1.5708 0 0"/>
           <geometry><box size="0.020 0.020 ${L1}"/></geometry>
           <material name="cfrp"/>
         </visual>
         <collision>
-          <origin xyz="${L1/2} 0 0" rpy="0 0 0"/>
-          <geometry><box size="${L1} 0.022 0.022"/></geometry>
+          <origin xyz="0 ${-L1/2} 0" rpy="0 0 0"/>
+          <geometry><box size="0.022 ${L1} 0.022"/></geometry>
         </collision>
       </xacro:unless>
       <inertial>
         <mass value="0.08"/>
-        <origin xyz="${L1/2} 0 0"/>
-        <inertia ixx="6.0e-6" ixy="0" ixz="0"
-                 iyy="2.2e-4" iyz="0" izz="2.2e-4"/>
-      </inertial>
-    </link>
-    <!-- ========== upper_arm_link -> forearm_link ========== -->
-    <!-- RMD-X6-60 | Y축 회전 (엘보우 피치), x=L1, Case C 오프셋 z=+18.8mm -->
+        <origin xyz="0 ${-L1/2} 0" rpy="0 0 0"/>
+        <inertia ixx="2.2e-4" ixy="0" ixz="0" iyy="6.0e-6" iyz="0" izz="2.2e-4"/>
+      </inertial>
+    </link>
+    <!-- ========== shoulder_link -> elbow_link (revolute, "엘보우 피치") ==========
+         [조인트] shoulder_lift_joint와 같은 이유로 axis는 X. 주축 오프셋은 -Y에서
+         +Z로 변경: L1(shoulder_link Y-extent)만큼 +Z로 이동 + Case C 보조
+         오프셋(off_elbow, +18.8mm)은 비게 된 Y자리로 옮겼다.
+         X축에는 off_gripper와 동일한 소치수 오프셋 적용.
+         [수정] Z축 180° 반전은 제거함 (shoulder_lift_joint 주석 참고 - 누적되면
+         링크마다 번갈아 뒤집혀서 pitch 축 방향이 어긋난다). -->
     <joint name="${prefix}elbow_joint" type="revolute">
-      <parent link="${prefix}upper_arm_link"/>
-      <child  link="${prefix}forearm_link"/>
-      <origin xyz="${L1} 0 ${off_elbow}" rpy="0 0 0"/>
-      <axis xyz="0 1 0"/>
-      <!-- 실측 인코더 리미트(raw_min/raw_max) - zero_offset. config/joint_calibration.yaml -->
-      <limit lower="${elbow_limit_lower}" upper="${elbow_limit_upper}"
-             effort="60.0" velocity="1.571"/>
-      <!-- RMD-X6-60 peak torque 60 Nm -->
+      <parent link="${prefix}shoulder_link"/>
+      <child  link="${prefix}elbow_link"/>
+      <origin xyz="-${off_gripper + off_elbow} 0 ${L1}" rpy="0 0 0"/>
+      <axis xyz="1 0 0"/>
+      <limit lower="${elbow_limit_lower}" upper="${elbow_limit_upper}" effort="60.0" velocity="1.571"/>
       <dynamics damping="0.5" friction="0.05"/>
     </joint>
-    <!-- forearm_link: CFRP 20x20x2T, L2 = 220mm -->
-    <link name="${prefix}forearm_link">
-      <xacro:if value="${use_mesh}">
-        <visual>
-          <origin xyz="0 0 0" rpy="0 0 0"/>
-          <!-- elbow_link.stl = RMD-X6-60 출력 플랜지 + L2 CFRP 튜브 + RMD-X4-36 케이스 통합 파츠
-               (실측 Y span 279.3mm ≈ RMD-X6-60 플랜지 + L2(220mm) + RMD-X4-36 케이스 두께, 일치) -->
+    <!-- elbow_link: RMD-X6-60 출력 플랜지 + L2 CFRP 튜브 + RMD-X4-36 케이스 통합 파츠 -->
+    <link name="${prefix}elbow_link">
+      <xacro:if value="${use_mesh}">
+        <!-- [시각화] X축 -90° 회전 적용. -->
+        <visual>
+          <origin xyz="0 0 0" rpy="${-pi/2} 0 0"/>
           <geometry><mesh filename="package://army_manipulator_description/meshes/visual/elbow_link.stl" scale="0.001 0.001 0.001"/></geometry>
           <material name="cfrp"/>
         </visual>
-        <collision>
-          <origin xyz="0 0 0" rpy="0 0 0"/>
+        <!-- [콜리전] visual과 동일 회전. -->
+        <collision>
+          <origin xyz="0 0 0" rpy="${-pi/2} 0 0"/>
           <geometry><mesh filename="package://army_manipulator_description/meshes/collision/elbow_link.stl" scale="0.001 0.001 0.001"/></geometry>
         </collision>
@@ -228,31 +237,31 @@
       <xacro:unless value="${use_mesh}">
         <visual>
-          <origin xyz="${L2/2} 0 0" rpy="0 1.5708 0"/>
+          <origin xyz="0 ${-L2/2} 0" rpy="1.5708 0 0"/>
           <geometry><box size="0.020 0.020 ${L2}"/></geometry>
           <material name="cfrp"/>
         </visual>
         <collision>
-          <origin xyz="${L2/2} 0 0" rpy="0 0 0"/>
-          <geometry><box size="${L2} 0.022 0.022"/></geometry>
+          <origin xyz="0 ${-L2/2} 0" rpy="0 0 0"/>
+          <geometry><box size="0.022 ${L2} 0.022"/></geometry>
         </collision>
       </xacro:unless>
       <inertial>
         <mass value="0.10"/>
-        <origin xyz="${L2/2} 0 0"/>
-        <inertia ixx="7.3e-6" ixy="0" ixz="0"
-                 iyy="4.0e-4" iyz="0" izz="4.0e-4"/>
-      </inertial>
-    </link>
-    <!-- ========== forearm_link -> wrist_link ========== -->
-    <!-- RMD-X4-36 | Y축 회전 (리스트 피치), x=L2, Case C 오프셋 z=-31.3mm -->
+        <origin xyz="0 ${-L2/2} 0"/>
+        <inertia ixx="4.0e-4" ixy="0" ixz="0" iyy="7.3e-6" iyz="0" izz="4.0e-4"/>
+      </inertial>
+    </link>
+    <!-- ========== elbow_link -> wrist_link (revolute, "리스트 피치") ==========
+         [조인트] 마찬가지로 axis X. 주축 오프셋은 -Y에서 +Z로 변경: L2(elbow_link
+         Y-extent)만큼 +Z로 이동 + Case C 보조 오프셋(off_wrist, -31.3mm)은 비게
+         된 Y자리로 옮겼다.
+         X축에는 off_gripper와 동일한 소치수 오프셋 적용.
+         [수정] Z축 180° 반전은 제거함 (shoulder_lift_joint 주석 참고). -->
     <joint name="${prefix}wrist_joint" type="revolute">
-      <parent link="${prefix}forearm_link"/>
+      <parent link="${prefix}elbow_link"/>
       <child  link="${prefix}wrist_link"/>
-      <origin xyz="${L2} 0 ${off_wrist}" rpy="0 0 0"/>
-      <axis xyz="0 1 0"/>
-      <!-- 실측 인코더 리미트(raw_min/raw_max) - zero_offset. config/joint_calibration.yaml -->
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