Commit message: WIP: rack-pinion gripper 관련 설정 및 launch 파일 정리

File: src/army_manipulator_description/urdf/army_manipulator_ros2_control.xacro (robot description, xacro)
@@ -8,5 +8,5 @@
   use_mock_hardware=false (팀원 Hardware Interface 완성 후)
     -> 버스별로 분리된 실제 플러그인을 사용:
-       - base_rotate_joint  : dynamixel_hardware/DynamixelHardware   (RS-485, XH540-W270-T)
+       - base_joint  : dynamixel_hardware/DynamixelHardware   (RS-485, XH540-W270-T)
        - gripper_joint      : dynamixel_hardware/DynamixelHardware   (TTL,   MX-106T)
        - shoulder/elbow/wrist : myactuator_rmd_hardware/MyActuatorRmdHardwareInterface (CAN, RMD-X8/X6/X4)
@@ -24,5 +24,5 @@
           <plugin>mock_components/GenericSystem</plugin>
         </hardware>
-        <joint name="${prefix}base_rotate_joint">
+        <joint name="${prefix}base_joint">
           <command_interface name="position"/>
           <state_interface name="position"><param name="initial_value">0.0</param></state_interface>
@@ -49,16 +49,33 @@
           <state_interface name="velocity"/>
         </joint>
+        <!-- rack_left_joint/rack_right_joint는 URDF에서 gripper_joint를 <mimic>하는
+             조인트다. 실측 결과 GenericSystem은 URDF의 <mimic> 태그를 자동으로
+             읽지 않고, <ros2_control><joint> 블록 안에 <param name="mimic">/
+             <param name="multiplier">를 직접 선언해야 그 값을 보고 gripper_joint
+             상태로부터 자동 계산해준다 (state_interface만 등록했을 때는 0.0으로
+             고정된 채 안 움직이는 것을 확인함). -->
+        <joint name="${prefix}rack_left_joint">
+          <param name="mimic">${prefix}gripper_joint</param>
+          <param name="multiplier">${pinion_pitch_radius}</param>
+          <state_interface name="position"><param name="initial_value">0.0</param></state_interface>
+          <state_interface name="velocity"/>
+        </joint>
+        <joint name="${prefix}rack_right_joint">
+          <param name="mimic">${prefix}gripper_joint</param>
+          <param name="multiplier">${-pinion_pitch_radius}</param>
+          <state_interface name="position"><param name="initial_value">0.0</param></state_interface>
+          <state_interface name="velocity"/>
+        </joint>
       </ros2_control>
     </xacro:if>
     <xacro:unless value="${use_mock_hardware}">
-      <!-- ===== base_rotate_joint : Dynamixel XH540-W270-T (RS-485) ===== -->
+      <!-- ===== base_joint : Dynamixel XH540-W270-T (TTL) ===== -->
       <ros2_control name="${prefix}base_bus" type="system">
         <hardware>
           <plugin>dynamixel_hardware/DynamixelHardware</plugin>
-          <!-- TODO: 실제 U2D2/RS-485 포트로 교체 -->
           <param name="usb_port">/dev/ttyUSB0</param>
           <param name="baud_rate">1000000</param>
         </hardware>
-        <joint name="${prefix}base_rotate_joint">
+        <joint name="${prefix}base_joint">
           <param name="id">1</param>
           <command_interface name="position"/>
@@ -87,5 +104,5 @@
           <plugin>myactuator_rmd_hardware/MyActuatorRmdHardwareInterface</plugin>
           <!-- TODO: 실제 CAN 인터페이스/ID/토크상수로 교체 -->
-          <param name="ifname">can1</param>
+          <param name="ifname">can_arm</param>
           <param name="actuator_id">4</param>
           <param name="torque_constant">1.0</param>
@@ -102,5 +119,5 @@
         <hardware>
           <plugin>myactuator_rmd_hardware/MyActuatorRmdHardwareInterface</plugin>
-          <param name="ifname">can1</param>
+          <param name="ifname">can_arm</param>
           <param name="actuator_id">5</param>
           <param name="torque_constant">1.0</param>
@@ -117,5 +134,5 @@
         <hardware>
           <plugin>myactuator_rmd_hardware/MyActuatorRmdHardwareInterface</plugin>
-          <param name="ifname">can1</param>
+          <param name="ifname">can_arm</param>
           <param name="actuator_id">6</param>
           <param name="torque_constant">1.0</param>
