Commit message: feat: add D455 supplybox grasp pipeline

File: src/army_manipulator_description/urdf/army_manipulator_ros2_control.xacro (robot description, xacro)
@@ -6,17 +6,18 @@
     -> mock_components/GenericSystem 로 5축 전부를 하나의 system 으로 노출.
        RViz + MoveIt2 플래닝 파이프라인 검증용.
-  use_mock_hardware=false (팀원 Hardware Interface 완성 후)
-    -> 버스별로 분리된 실제 플러그인을 사용:
-       - base_joint  : dynamixel_hardware/DynamixelHardware   (RS-485, XH540-W270-T)
-       - gripper_joint      : dynamixel_hardware/DynamixelHardware   (TTL,   MX-106T)
-       - shoulder/elbow/wrist : myactuator_rmd_hardware/MyActuatorRmdHardwareInterface (CAN, RMD-X8/X6/X4)
-       plugin 이름/파라미터는 각각
-       https://github.com/dynamixel-community/dynamixel_hardware ,
-       https://github.com/2b-t/myactuator_rmd_ros (myactuator_rmd_hardware) 기준.
-       usb_port / ifname / actuator_id 는 실장비 배선 확정 후 팀원과 맞춰서 수정할 것.
+  use_mock_hardware=false (실제 하드웨어)
+    -> dolbotZ(9o9hz/dolbotZ)에서 검증된 플러그인/파라미터 구조를 그대로 이식:
+       - base_joint + gripper_joint : dynamixel_hardware_interface/DynamixelHardware
+         (하나의 system, TTL 버스 하나에 ID로 구분. gripper=ID4, base=ID0 실측값)
+       - shoulder/elbow/wrist       : rmd_hardware_interface/MyActuatorRmdHardwareInterface
+         (CAN, 조인트당 개별 actuator 블록)
   ============================================================
 -->
 <robot xmlns:xacro="http://www.ros.org/wiki/xacro">
   <xacro:macro name="army_manipulator_ros2_control" params="prefix use_mock_hardware">
+    <xacro:arg name="dxl_port_name" default="/dev/ttyUSB0"/>
+    <xacro:arg name="dxl_baud_rate" default="57600"/>
+    <xacro:arg name="rmd_ifname" default="can_arm"/>
+    <xacro:arg name="rmd_timeout" default="100"/>
     <xacro:if value="${use_mock_hardware}">
       <ros2_control name="${prefix}army_manipulator_system" type="system">
@@ -49,10 +50,4 @@
           <state_interface name="velocity"/>
         </joint>
-        <!-- rack_left_joint/rack_right_joint는 URDF에서 gripper_joint를 <mimic>하는
-             조인트다. 실측 결과 GenericSystem은 URDF의 <mimic> 태그를 자동으로
-             읽지 않고, <ros2_control><joint> 블록 안에 <param name="mimic">/
-             <param name="multiplier">를 직접 선언해야 그 값을 보고 gripper_joint
-             상태로부터 자동 계산해준다 (state_interface만 등록했을 때는 0.0으로
-             고정된 채 안 움직이는 것을 확인함). -->
         <joint name="${prefix}rack_left_joint">
           <param name="mimic">${prefix}gripper_joint</param>
@@ -70,74 +65,135 @@
     </xacro:if>
     <xacro:unless value="${use_mock_hardware}">
-      <!-- ===== base_joint : Dynamixel XH540-W270-T (TTL) ===== -->
-      <ros2_control name="${prefix}base_bus" type="system">
-        <hardware>
-          <plugin>dynamixel_hardware/DynamixelHardware</plugin>
-          <param name="usb_port">/dev/ttyUSB0</param>
-          <param name="baud_rate">1000000</param>
-        </hardware>
+      <!-- ===== base_joint(XH540, ID0) + gripper_joint(MX-106T, ID4) : 하나의 TTL 버스 ===== -->
+      <ros2_control name="${prefix}dynamixel_system" type="system">
+        <hardware>
+          <plugin>dynamixel_hardware_interface/DynamixelHardware</plugin>
+          <param name="port_name">$(arg dxl_port_name)</param>
+          <param name="baud_rate">$(arg dxl_baud_rate)</param>
+          <param name="dynamixel_model_folder">/param/dxl_model</param>
+          <param name="number_of_joints">2</param>
+          <param name="number_of_transmissions">2</param>
+          <param name="disable_torque_at_init">true</param>
+          <param name="error_timeout_ms">1000</param>
+          <param name="transmission_to_joint_matrix">1,0,0,1</param>
+          <param name="joint_to_transmission_matrix">1,0,0,1</param>
+          <param name="dynamixel_state_pub_msg_name">dynamixel_hardware_interface/dxl_state</param>
+          <param name="get_dynamixel_data_srv_name">dynamixel_hardware_interface/get_dxl_data</param>
+          <param name="set_dynamixel_data_srv_name">dynamixel_hardware_interface/set_dxl_data</param>
+          <param name="reboot_dxl_srv_name">dynamixel_hardware_interface/reboot_dxl</param>
+          <param name="set_dxl_torque_srv_name">dynamixel_hardware_interface/set_dxl_torque</param>
+        </hardware>
+        <!-- joint/gpio 순서가 transmission_to_joint_matrix(항등행렬)로 1:1 매핑되므로
+             순서를 반드시 gripper -> base 로 맞춘다 (dolbotZ 실측 순서와 동일). -->
+        <joint name="${prefix}gripper_joint">
+          <command_interface name="position"/>
+          <state_interface name="position"/>
+          <state_interface name="velocity"/>
+          <state_interface name="effort"/>
+        </joint>
         <joint name="${prefix}base_joint">
-          <param name="id">1</param>
-          <command_interface name="position"/>
-          <state_interface name="position"/>
-          <state_interface name="velocity"/>
-        </joint>
-      </ros2_control>
-      <!-- ===== gripper_joint : Dynamixel MX-106T (TTL) ===== -->
-      <ros2_control name="${prefix}gripper_bus" type="system">
-        <hardware>
-          <plugin>dynamixel_hardware/DynamixelHardware</plugin>
-          <!-- TODO: 실제 U2D2/TTL 포트로 교체 -->
-          <param name="usb_port">/dev/ttyUSB1</param>
-          <param name="baud_rate">1000000</param>
-        </hardware>
-        <joint name="${prefix}gripper_joint">
-          <param name="id">5</param>
-          <command_interface name="position"/>
-          <state_interface name="position"/>
-          <state_interface name="velocity"/>
-        </joint>
-      </ros2_control>
-      <!-- ===== shoulder_lift_joint : RMD-X8-120 (CAN) ===== -->
+          <command_interface name="position"/>
+          <state_interface name="position"/>
+          <state_interface name="velocity"/>
+          <state_interface name="effort"/>
+        </joint>
+        <gpio name="dxl1">
+          <param name="type">dxl</param>
+          <param name="ID">4</param>
+          <command_interface name="Goal Position"/>
+          <state_interface name="Present Position"/>
+          <state_interface name="Present Velocity"/>
+          <state_interface name="Present Current"/>
+          <state_interface name="Torque Enable"/>
+          <state_interface name="Hardware Error Status"/>
+          <param name="Return Delay Time">0</param>
+        </gpio>
+        <gpio name="dxl2">
+          <param name="type">dxl</param>
+          <param name="ID">0</param>
+          <command_interface name="Goal Position"/>
+          <state_interface name="Present Position"/>
+          <state_interface name="Present Velocity"/>
+          <state_interface name="Present Current"/>
+          <state_interface name="Torque Enable"/>
+          <state_interface name="Hardware Error Status"/>
+          <param name="Return Delay Time">0</param>
+        </gpio>
+      </ros2_control>
+      <!-- ===== shoulder_lift_joint : RMD-X8-120 (CAN, ID4) ===== -->
       <ros2_control name="${prefix}shoulder_actuator" type="actuator">
         <hardware>
-          <plugin>myactuator_rmd_hardware/MyActuatorRmdHardwareInterface</plugin>
-          <!-- TODO: 실제 CAN 인터페이스/ID/토크상수로 교체 -->
-          <param name="ifname">can_arm</param>
+          <plugin>rmd_hardware_interface/MyActuatorRmdHardwareInterface</plugin>
+          <param name="ifname">$(arg rmd_ifname)</param>
           <param name="actuator_id">4</param>
+          <!-- TODO(rmd-tuning): torque_constant/max_velocity/current 관련 값은
+               RMD-X8-120 데이터시트 기준 임시값. 실측 후 조정 필요. -->
           <param name="torque_constant">1.0</param>
+          <param name="max_velocity">1.047</param>
+          <param name="velocity_alpha">0.1</param>
+          <param name="effort_alpha">0.1</param>
+          <param name="software_current_limit">10.0</param>
+          <param name="current_release_threshold">8.0</param>
+          <param name="current_limit_duration_ms">50</param>
+          <param name="current_retreat_velocity">0.1</param>
+          <param name="current_max_retreat_distance">0.174533</param>
+          <param name="timeout">$(arg rmd_timeout)</param>
         </hardware>
         <joint name="${prefix}shoulder_lift_joint">
           <command_interface name="position"/>
-          <state_interface name="position"/>
-          <state_interface name="velocity"/>
-          <state_interface name="effort"/>
-        </joint>
-      </ros2_control>
-      <!-- ===== elbow_joint : RMD-X6-60 (CAN) ===== -->
+          <command_interface name="velocity"/>
+          <command_interface name="effort"/>
+          <state_interface name="position"/>
+          <state_interface name="velocity"/>
+          <state_interface name="effort"/>
+        </joint>
+      </ros2_control>
+      <!-- ===== elbow_joint : RMD-X6-60 (CAN, ID5) ===== -->
       <ros2_control name="${prefix}elbow_actuator" type="actuator">
         <hardware>
-          <plugin>myactuator_rmd_hardware/MyActuatorRmdHardwareInterface</plugin>
-          <param name="ifname">can_arm</param>
+          <plugin>rmd_hardware_interface/MyActuatorRmdHardwareInterface</plugin>
+          <param name="ifname">$(arg rmd_ifname)</param>
           <param name="actuator_id">5</param>
           <param name="torque_constant">1.0</param>
+          <param name="max_velocity">1.571</param>
+          <param name="velocity_alpha">0.1</param>
+          <param name="effort_alpha">0.1</param>
+          <param name="software_current_limit">10.0</param>
+          <param name="current_release_threshold">8.0</param>
+          <param name="current_limit_duration_ms">50</param>
+          <param name="current_retreat_velocity">0.1</param>
+          <param name="current_max_retreat_distance">0.174533</param>
+          <param name="timeout">$(arg rmd_timeout)</param>
         </hardware>
         <joint name="${prefix}elbow_joint">
           <command_interface name="position"/>
-          <state_interface name="position"/>
-          <state_interface name="velocity"/>
-          <state_interface name="effort"/>
-        </joint>
-      </ros2_control>
-      <!-- ===== wrist_joint : RMD-X4-36 (CAN) ===== -->
+          <command_interface name="velocity"/>
+          <command_interface name="effort"/>
+          <state_interface name="position"/>
+          <state_interface name="velocity"/>
+          <state_interface name="effort"/>
+        </joint>
+      </ros2_control>
+      <!-- ===== wrist_joint : RMD-X4-36 (CAN, ID6) ===== -->
       <ros2_control name="${prefix}wrist_actuator" type="actuator">
         <hardware>
-          <plugin>myactuator_rmd_hardware/MyActuatorRmdHardwareInterface</plugin>
-          <param name="ifname">can_arm</param>
+          <plugin>rmd_hardware_interface/MyActuatorRmdHardwareInterface</plugin>
+          <param name="ifname">$(arg rmd_ifname)</param>
           <param name="actuator_id">6</param>
           <param name="torque_constant">1.0</param>
+          <param name="max_velocity">2.618</param>
+          <param name="velocity_alpha">0.1</param>
+          <param name="effort_alpha">0.1</param>
+          <param name="software_current_limit">10.0</param>
+          <param name="current_release_threshold">8.0</param>
+          <param name="current_limit_duration_ms">50</param>
+          <param name="current_retreat_velocity">0.1</param>
+          <param name="current_max_retreat_distance">0.174533</param>
+          <param name="timeout">$(arg rmd_timeout)</param>
         </hardware>
         <joint name="${prefix}wrist_joint">
           <command_interface name="position"/>
+          <command_interface name="velocity"/>
+          <command_interface name="effort"/>
           <state_interface name="position"/>
           <state_interface name="velocity"/>

Commit message: Sync arm packages from dolbotZ

File: src/army_manipulator_description/urdf/army_manipulator.urdf.xacro (robot description, xacro)
@@ -9,4 +9,99 @@
   <xacro:include filename="$(find army_manipulator_description)/urdf/army_manipulator_macro.xacro"/>
   <link name="world"/>
-  <xacro:army_manipulator prefix="" parent="world" use_mock_hardware="$(arg use_mock_hardware)" use_mesh="$(arg use_mesh)"/>
+  <!-- ========== 차체(chassis) 충돌 지오메트리 ==========
+       [추가] R3 "차체 간섭 방지" 요구사항용. 이 전까지는 planning scene에
+       차체가 아예 없어서 MoveIt이 팔-차체 충돌을 원천적으로 못 봤다
+       (자기충돌 체크는 SRDF disable_collisions로 팔 링크끼리만 되어있었음).
+       2026-08-24 실측값 반영. 박스 중심은 차체 지면 접촉면 중앙, 팔은 박스
+       윗면에서 (mount_x, mount_y) 만큼 이동하고 거기서 mount_z 만큼 더 위로
+       올라간 위치(마운트 브라켓 높이)에 장착된다고 가정. mount_x는 ROS 표준
+       관례(+x=전방)를 가정한 값 — 실제 로봇 정면 방향이 다르면 부호를
+       바꿀 것. 좌우(mount_y) 오프셋은 실측 안 돼 중앙(0.0)으로 둠. 값이
+       또 바뀌면 launch argument로 덮어쓰면 된다(코드 수정 불필요):
+         ros2 launch ... chassis_length:=... chassis_width:=...
+         chassis_height:=... chassis_mount_x:=... chassis_mount_y:=...
+         chassis_mount_z:=... -->
+  <xacro:arg name="chassis_length" default="0.78"/>
+  <xacro:arg name="chassis_width" default="0.50"/>
+  <xacro:arg name="chassis_height" default="0.30"/>
+  <xacro:arg name="chassis_mount_x" default="0.25"/>
+  <xacro:arg name="chassis_mount_y" default="0.0"/>
+  <!-- 차체 상단(0.30m)과 팔 실제 장착 높이(바닥 기준 0.35m) 사이 0.05m 브라켓 높이 -->
+  <xacro:arg name="chassis_mount_z" default="0.05"/>
+  <!-- ========== 차체 위 세로 프레임(20x20 프로파일, 2026-08-31 실측 갱신) ==========
+       robot.stl(636,838 tri)을 collision에 그대로 쓰면 move_group이 멎어서
+       (위 기록 참고) 간섭 계산이 실제로 필요한 부분만 박스로 근사한다.
+       world 원점(z=0, 바닥) 기준, 전방 x=90.461mm 위치에서 양옆
+       (y=±chassis_width/2)으로 기둥 2개가 z=920.188mm(=805.188+115mm 보정,
+       2026-08-30)까지 올라간다.
+       가로대(crossbar): 2026-08-31 실측으로 갱신 - 차체 상단(chassis_height=
+       300mm)에서 530mm 위(=바닥 기준 830mm)가 20x20 프로파일의 아래쪽 면,
+       거기서 20mm를 더한 850mm(바닥 기준)가 위쪽 면 -> 중심은 바닥 기준
+       840mm. x위치는 기둥과 동일(변경 없음). -->
+  <xacro:property name="frame_post_x"      value="0.090461"/>
+  <xacro:property name="frame_post_y"      value="${$(arg chassis_width) / 2.0}"/>
+  <xacro:property name="frame_post_height" value="0.920188"/>
+  <xacro:property name="frame_crossbar_z"  value="0.840"/>
+  <xacro:property name="frame_profile"     value="0.020"/>
+  <joint name="world_to_chassis" type="fixed">
+    <parent link="world"/>
+    <child link="chassis_link"/>
+    <origin xyz="0 0 0" rpy="0 0 0"/>
+  </joint>
+  <link name="chassis_link">
+    <visual>
+      <origin xyz="0 0 ${$(arg chassis_height) / 2.0}" rpy="0 0 0"/>
+      <geometry><box size="$(arg chassis_length) $(arg chassis_width) $(arg chassis_height)"/></geometry>
+      <material name="motor_dark"/>
+    </visual>
+    <collision>
+      <origin xyz="0 0 ${$(arg chassis_height) / 2.0}" rpy="0 0 0"/>
+      <geometry><box size="$(arg chassis_length) $(arg chassis_width) $(arg chassis_height)"/></geometry>
+    </collision>
+    <visual>
+      <origin xyz="${frame_post_x} ${frame_post_y} ${frame_post_height / 2.0}" rpy="0 0 0"/>
+      <geometry><box size="${frame_profile} ${frame_profile} ${frame_post_height}"/></geometry>
+      <material name="motor_dark"/>
+    </visual>
+    <collision>
+      <origin xyz="${frame_post_x} ${frame_post_y} ${frame_post_height / 2.0}" rpy="0 0 0"/>
+      <geometry><box size="${frame_profile} ${frame_profile} ${frame_post_height}"/></geometry>
+    </collision>
+    <visual>
+      <origin xyz="${frame_post_x} ${-frame_post_y} ${frame_post_height / 2.0}" rpy="0 0 0"/>
+      <geometry><box size="${frame_profile} ${frame_profile} ${frame_post_height}"/></geometry>
+      <material name="motor_dark"/>
+    </visual>
+    <collision>
+      <origin xyz="${frame_post_x} ${-frame_post_y} ${frame_post_height / 2.0}" rpy="0 0 0"/>
+      <geometry><box size="${frame_profile} ${frame_profile} ${frame_post_height}"/></geometry>
+    </collision>
+    <visual>
+      <origin xyz="${frame_post_x} 0 ${frame_crossbar_z}" rpy="0 0 0"/>
+      <geometry><box size="${frame_profile} $(arg chassis_width) ${frame_profile}"/></geometry>
+      <material name="motor_dark"/>
+    </visual>
+    <collision>
+      <origin xyz="${frame_post_x} 0 ${frame_crossbar_z}" rpy="0 0 0"/>
+      <geometry><box size="${frame_profile} $(arg chassis_width) ${frame_profile}"/></geometry>
+    </collision>
+    <inertial>
+      <!-- 차체는 고정(fixed) 링크라 관성값이 플래닝/제어에 안 쓰이지만,
+           URDF 파서가 링크에 관성 없이 collision만 있으면 경고를 내는 경우가
+           있어 형식상 채워둔다. -->
+      <mass value="1.0"/>
+      <origin xyz="0 0 0"/>
+      <inertia ixx="0.05" ixy="0" ixz="0" iyy="0.05" iyz="0" izz="0.05"/>
+    </inertial>
+  </link>
+  <joint name="chassis_to_arm_mount" type="fixed">
+    <parent link="chassis_link"/>
+    <child link="arm_mount_link"/>
+    <!-- chassis_link 원점이 이제 world 지면(z=0, world_to_chassis 참고)이라
+         차체 상단(chassis_height) + 브라켓 높이(chassis_mount_z)를 그대로
+         더해야 문서화된 팔 마운트 높이(바닥 기준 0.35m)가 나온다. -->
+    <origin xyz="$(arg chassis_mount_x) $(arg chassis_mount_y) ${$(arg chassis_height) + $(arg chassis_mount_z)}" rpy="0 0 0"/>
+  </joint>
+  <link name="arm_mount_link"/>
+  <xacro:army_manipulator prefix="" parent="arm_mount_link" use_mock_hardware="$(arg use_mock_hardware)" use_mesh="$(arg use_mesh)"/>
 </robot>
